File: MicroPad/_autosave-MicroPad.kicad_sch (KiCad schematic)
At the start: 68 parts, among them J10 Conn_01x02, J11 Conn_01x02, J12 Conn_01x02, J2 USB_C_Receptacle_USB2.0_16P, J4 Programming header, J5 SPI for E-Ink Display, J6 B2B-PH-K-S (Battery), J9 Conn_01x02, SW1 RESET, SW10 SWITCH, SW11 SWITCH, SW13 SWITCH, SW14 SWITCH, SW15 RotaryEncoder_Switch_MP, SW2 BOOT, SW3 SWITCH, SW4 SWITCH, SW5 SWITCH, SW6 SWITCH, SW7 SWITCH, SW8 SWITCH, SW9 SWITCH, U1 BQ24075RGT, U3 ESP32-S3-WROOM-1, U5 ESD7104MUTAG, U6 AP2112K-3.3

Commit message: new version with bigger display and one key less
Connections:
- net CS: now also U3.12 (IO8); no longer U3.8 (IO15)
- no-connect marks 9 -> 17
Changed lines of the file:
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@@
+	)
+	(no_connect
+		(at 133.35 110.49)
 	)
 	(no_connect
@@
 	)
 	(no_connect
+		(at 163.83 72.39)
+	)
+	(no_connect
 		(at 163.83 87.63)
+	)
+	(no_connect
+		(at 133.35 82.55)
+	)
+	(no_connect
+		(at 133.35 90.17)
+	)
+	(no_connect
+		(at 133.35 113.03)
+	)
+	(no_connect
+		(at 133.35 87.63)
+	)
+	(no_connect
+		(at 163.83 74.93)
 	)
 	(no_connect
@@
 		(at 102.87 64.77)
 	)
+	(no_connect
+		(at 133.35 85.09)
+	)
 	(wire
 		(pts
@@
 	(wire
 		(pts
-			(xy 130.81 110.49) (xy 133.35 110.49)
-		)
-		(stroke
-			(width 0)
-			(type default)
-		)
-	)
-	(wire
-		(pts
 			(xy 45.72 30.48) (xy 48.26 30.48)
 		)
@@
 		(pts
 			(xy 26.67 121.92) (xy 39.37 121.92)
+		)
+		(stroke
+			(width 0)
+			(type default)
+		)
+	)
+	(wire
+		(pts
+			(xy 129.54 92.71) (xy 133.35 92.71)
 		)
 		(stroke
@@
 		)
 	)
+	(label "CS"
+		(at 129.54 92.71 180)
+		(effects
+			(font
+				(size 1.27 1.27)
+			)
+			(justify right bottom)
+		)
+	)
 	(label "USB_D-"
 		(at 50.8 36.83 0)
@@
 		(effects
 			(font
-				(size 1.27 1.27)
-			)
-			(justify right bottom)
-		)
-	)
-	(label "CS"
-		(at 130.81 110.49 180)
-		(effects
-			(font
