File: MicroPad/MicroPad.kicad_sch (KiCad schematic)
At the start: 68 parts, among them J10 Conn_01x02, J11 Conn_01x02, J12 Conn_01x02, J2 USB_C_Receptacle_USB2.0_16P, J4 Programming header, J5 SPI for E-Ink Display, J6 B2B-PH-K-S (Battery), J9 Conn_01x02, SW1 RESET, SW10 SWITCH, SW11 SWITCH, SW13 SWITCH, SW14 SWITCH, SW15 RotaryEncoder_Switch_MP, SW2 BOOT, SW3 SWITCH, SW4 SWITCH, SW5 SWITCH, SW6 SWITCH, SW7 SWITCH, SW8 SWITCH, SW9 SWITCH, U1 BQ24075RGT, U3 ESP32-S3-WROOM-1, U5 ESD7104MUTAG, U6 AP2112K-3.3

Commit message: new version
Parts:
- removed U5: ESD7104MUTAG, ESD7104MUTAG:IC_ESD7104MUTAG, symbol ESD7104MUTAG:ESD7104MUTAG
- added C1: 220u, Capacitor_SMD:CP_Elec_6.3x7.7, symbol Device:C_Polarized
- added C15: 100n, Capacitor_SMD:C_0805_2012Metric_Pad1.18x1.45mm_HandSolder, symbol Device:C
- added U2: USBLC6-2SC6, Package_TO_SOT_SMD:SOT-23-6, symbol Power_Protection:USBLC6-2SC6
Connections:
- net +3V3: now also C1.1
- net CS: now also U3.12 (IO8); no longer U3.8 (IO15)
- net GND: now also C1.2, C15.2, U2.2 (GND)
- net USB_D+: now also U2.4 (I/O2); no longer J2.A6 (D+), J2.B6 (D+)
- net USB_D-: now also U2.6 (I/O1); no longer J2.A7 (D-), J2.B7 (D-)
- net VBUS: now also C15.1, U2.5 (VBUS)
- net S1 renamed Diode out
- new net D+: J2.A6 (D+), J2.B6 (D+), U2.3 (I/O2)
- new net D-: J2.A7 (D-), J2.B7 (D-), U2.1 (I/O1)
- no-connect marks 9 -> 18
Other:
- note added: "PWR FLAG(s)"

Commit message: new version
Other:
- note added: "E-Ink SPI"
- note removed: "E-Ink"
- company: (none) -> Jonas Lindinger
- title: (none) -> Micro Pad
Changed lines of the file:
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@@
 	(generator_version "10.0")
 	(paper "A4")
+	(title_block
+		(title "Micro Pad")
+		(date "2026-04-24")
+		(rev "v1")
+		(company "Jonas Lindinger")
+	)
 	(rectangle
 		(start 87.63 119.38)
@@
 		)
 	)
-	(text "E-Ink"
-		(exclude_from_sim no)
-		(at 180.594 39.878 0)
-		(effects
-			(font
+	(text "E-Ink SPI"
+		(exclude_from_sim no)
+		(at 182.372 39.37 0)
+		(effects
+			(font

Commit message: add: new version
Parts:
- removed SW15: RotaryEncoder_Switch_MP, Rotary_Encoder:RotaryEncoder_Alps_EC11E-Switch_Vertical_H20mm_MountingHoles, symbol Device:RotaryEncoder_Switch_MP
- added SW12: RotaryEncoder_Switch, Rotary_Encoder:RotaryEncoder_Alps_EC11E-Switch_Vertical_H20mm, symbol Device:RotaryEncoder_Switch
Connections:
- net A: now also SW12.A
- net B: now also SW12.B
- net C4: now also SW12.S2
- net Diode out: now also SW12.S1
- net GND: now also SW12.C
- no-connect marks 18 -> 17
Changed lines of the file:
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@@
 	)
 	(no_connect
-		(at 102.87 64.77)
-	)
-	(no_connect
 		(at 133.35 85.09)
 	)
@@
 	(wire
 		(pts
+			(xy 116.84 54.61) (xy 110.49 54.61)
+		)
+		(stroke
+			(width 0)
+			(type default)
+		)
+	)
+	(wire
+		(pts
 			(xy 54.61 76.2) (xy 54.61 101.6)
 		)
@@
 	(wire
 		(pts
+			(xy 92.71 54.61) (xy 95.25 54.61)
+		)
+		(stroke
+			(width 0)
+			(type default)
+		)
+	)
+	(wire
+		(pts
 			(xy 38.1 160.02) (xy 25.4 160.02)
 		)
@@
 	(wire
 		(pts
+			(xy 111.76 59.69) (xy 110.49 59.69)
+		)
+		(stroke
+			(width 0)
+			(type default)
+		)
+	)
+	(wire
+		(pts
 			(xy 160.02 157.48) (xy 160.02 154.94)
 		)
@@
 	(wire
 		(pts
+			(xy 92.71 59.69) (xy 95.25 59.69)
+		)
+		(stroke
+			(width 0)
+			(type default)
+		)
+	)
+	(wire
+		(pts
 			(xy 166.37 80.01) (xy 163.83 80.01)
 		)
@@
 	)
 	(label "C4"
-		(at 110.49 59.69 0)
+		(at 111.76 59.69 0)
 		(effects
 			(font
@@
 	)
 	(label "A"
-		(at 95.25 54.61 180)
+		(at 92.71 54.61 180)
 		(effects
 			(font
@@
 	)
 	(label "B"
-		(at 95.25 59.69 180)
+		(at 92.71 59.69 180)
 		(effects
 			(font
@@
 	)
 	(label "Diode out"
-		(at 110.49 54.61 0)
+		(at 116.84 54.61 270)
 		(effects
 			(font
 				(size 1.27 1.27)
 			)
-			(justify left bottom)
+			(justify right bottom)
 		)
 	)
@@
 	)
 	(symbol
+		(lib_id "Device:RotaryEncoder_Switch")
+		(at 102.87 57.15 0)
+		(unit 1)
+		(body_style 1)
+		(exclude_from_sim no)
+		(in_bom yes)
+		(on_board yes)
+		(in_pos_files yes)
+		(dnp no)
+		(fields_autoplaced yes)
+		(property "Reference" "SW12"
+			(at 102.87 46.99 0)
+			(show_name no)
+			(do_not_autoplace no)
+			(effects
+				(font
+					(size 1.27 1.27)
+				)
+			)
+		)
+		(property "Value" "RotaryEncoder_Switch"
+			(at 102.87 49.53 0)
+			(show_name no)
+			(do_not_autoplace no)
+			(effects
+				(font
+					(size 1.27 1.27)
+				)
+			)
+		)
+		(property "Footprint" "Rotary_Encoder:RotaryEncoder_Alps_EC11E-Switch_Vertical_H20mm"
+			(at 99.06 53.086 0)
+			(hide yes)
+			(show_name no)
+			(do_not_autoplace no)
+			(effects
+				(font
+					(size 1.27 1.27)
+				)
+			)
+		)
+		(property "Datasheet" ""
+			(at 102.87 50.546 0)
+			(hide yes)
+			(show_name no)
+			(do_not_autoplace no)
+			(effects
+				(font
+					(size 1.27 1.27)
+				)
+			)
+		)
+		(property "Description" "Rotary encoder, dual channel, incremental quadrate outputs, with switch"
+			(at 102.87 57.15 0)
+			(hide yes)
+			(show_name no)
+			(do_not_autoplace no)
+			(effects
+				(font
+					(size 1.27 1.27)
+				)
+			)
+		)
+		(pin "S1"
+		)
+		(pin "C"
+		)
+		(pin "S2"
+		)
+		(pin "A"
+		)
+		(pin "B"
+		)
+		(instances
+			(project "MicroPad"
+				(path "/004cc7b8-7c24-4edb-87f9-f7a29ef0ea7f"
+					(reference "SW12")
+					(unit 1)
+				)
+			)
+		)
+	)
+	(symbol
 		(lib_id "Device:D")
 		(at 64.77 118.11 270)
@@
 	)
 	(symbol
-		(lib_id "Device:RotaryEncoder_Switch_MP")
-		(at 102.87 57.15 0)
-		(unit 1)
-		(body_style 1)
-		(exclude_from_sim no)
-		(in_bom yes)
-		(on_board yes)
-		(in_pos_files yes)
-		(dnp no)
-		(fields_autoplaced yes)
-		(property "Reference" "SW15"
-			(at 102.87 46.99 0)
-			(show_name no)
-			(do_not_autoplace no)
-			(effects
-				(font
-					(size 1.27 1.27)
-				)
-			)
-		)
-		(property "Value" "RotaryEncoder_Switch_MP"
-			(at 102.87 49.53 0)
-			(show_name no)
-			(do_not_autoplace no)
-			(effects
-				(font
-					(size 1.27 1.27)
-				)
-			)
-		)
-		(property "Footprint" "Rotary_Encoder:RotaryEncoder_Alps_EC11E-Switch_Vertical_H20mm_MountingHoles"
-			(at 99.06 53.086 0)
-			(hide yes)
-			(show_name no)
-			(do_not_autoplace no)
-			(effects
-				(font
-					(size 1.27 1.27)
-				)
-			)
-		)
-		(property "Datasheet" ""
-			(at 102.87 69.85 0)
-			(hide yes)
-			(show_name no)
-			(do_not_autoplace no)
-			(effects
-				(font
-					(size 1.27 1.27)
-				)
-			)
-		)
-		(property "Description" "Rotary encoder, dual channel, incremental quadrate outputs, with switch and MP Pin"
-			(at 102.87 72.39 0)
-			(hide yes)
-			(show_name no)
-			(do_not_autoplace no)
-			(effects
-				(font
-					(size 1.27 1.27)
-				)
-			)
-		)
-		(pin "C"
-		)
-		(pin "S1"
-		)
-		(pin "B"
-		)
-		(pin "A"
-		)
-		(pin "MP"
-		)
-		(pin "S2"
-		)
-		(instances
-			(project "MicroPad"
-				(path "/004cc7b8-7c24-4edb-87f9-f7a29ef0ea7f"
-					(reference "SW15")
-					(unit 1)
-				)
-			)
-		)
-	)
-	(symbol
 		(lib_id "power:GND")
 		(at 82.55 144.78 180)
@@
 		(dnp no)
 		(property "Reference" "C15"
-			(at 105.664 15.494 90)
+			(at 104.648 15.748 90)
 			(show_name no)
 			(do_not_autoplace no)

Commit message: new version
Parts:
- added S1: 500ASSP1SM6QE, 500ASSP1SM6QE:SW_500ASSP1SM6QE, symbol 500ASSP1SM6QE:500ASSP1SM6QE
Connections:
- net PWR OUT renamed PWR S1
- net PWR S1: now also S1.2; no longer C14.2, U6.1 (VIN), U6.3 (EN)
- new net PWR S2: C14.2, S1.1, U6.1 (VIN), U6.3 (EN)
- no-connect marks 17 -> 18
